File: home-robot-r1/pcb/r1_power_io.kicad_sch (KiCad schematic)
At the start: 73 parts, among them J1 Battery in, J10 Bumper L, J11 Bumper R, J12 Arm button, J13 Motor toggle loop, J14 Spare I2C, J15 Spare GPIO, J2 Master rocker, J3 Jetson 5V, J4 Left motor, J5 Right motor, J6 Cliff 1, J7 Cliff 2, J8 Cliff 3, J9 Cliff 4, K1 G5LE-1 DC5, Q1 2N7002, Q2 2N7002, Q3 2N7002, Q4 2N7002, Q5 2N7002, U1A Pico left row, U1B Pico right row, U2 GY-521 MPU-6050, U3L DRV8874 left, VM/EN/PH row, U3P DRV8874 left, VIN/OUT row, U4L DRV8874 right, VM/EN/PH row, U4P DRV8874 right, VIN/OUT row, U5A Regulator in (P03 module), U5B Regulator out (P03 module)

Commit message: Sync: bay B12a connectors, B12b sim cleanups, task G bumper recovery
R1 from power-io-board 8bd8195:
- Battery, rocker and Jetson connectors that can't be swapped (J1 XT30, J2 VH, J3 Micro-Fit):
  board re-placed and re-routed, power check, fab files, CAD and harness updated.
- Final-review guide fixes (BRINGUP, ORDERING, pigtail lengths) and test cleanups.

Simulator from main 94d346d:
- Statistical scenario checks, IMU minors, C++/comment minors (B12b).
- Contact recovery with no straight trail behind the robot: re-planned back-off, slow creep
  over driven ground, then a 60 s cap and a stop message (task G).
- 2D house harness (tests/house2d), mapping analysis and the Unreal contact replay.
- docs/WORKFLOW.md: one task = one branch, one thread.

Co-Authored-By: Claude Opus 5.5 <noreply@anthropic.com>
Parts:
- J1: footprint Connector_JST:JST_VH_B2P-VH_1x02_P3.96mm_Vertical -> Connector_AMASS:AMASS_XT30UPB-M_1x02_P5.0mm_Vertical
- J3: footprint Connector_JST:JST_VH_B2P-VH_1x02_P3.96mm_Vertical -> Connector_Molex:Molex_Micro-Fit_3.0_43650-0200_1x02_P3.00mm_Horizontal
Changed lines of the file:
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@@
 			)
 		)
-		(property "Footprint" "Connector_JST:JST_VH_B2P-VH_1x02_P3.96mm_Vertical"
+		(property "Footprint" "Connector_AMASS:AMASS_XT30UPB-M_1x02_P5.0mm_Vertical"
 			(at 228.6 88.9 0)
 			(effects
@@
 			)
 		)
-		(property "Footprint" "Connector_JST:JST_VH_B2P-VH_1x02_P3.96mm_Vertical"
+		(property "Footprint" "Connector_Molex:Molex_Micro-Fit_3.0_43650-0200_1x02_P3.00mm_Horizontal"
 			(at 228.6 152.4 0)
 			(effects

Commit message: Board changes before fab: CS RC filters, DNP VSYS diode, ARM pull-up, 10k I2C pull-ups, 0.3 mm LP12 vias, JLCPCB DRC rules (LIO-226)
- CS filters: R24 / R25 (4.7k) + C4 / C5 (100 nF, LP12 GND vias) on new nets L_CS_ADC / R_CS_ADC
  (GP27 / GP28, RC 0.47 ms), placed beside the drivers' CS pins: both Pico columns are full at
  the silk-label pitch, so there is no legal 0805 spot by U1B.7 / U1B.9.
- D2: SS14 (SMA, DNP) from 5V to a new VSYS net at the Pico's pin 39 (U1B.2); VSYS left NC.
  The only legal SMA spot is the north end of DRV_R's interior.
- R26: 10k ARM pull-up at the foot of the U1A column, with a notch in the VBAT_SW F.Cu strip
  (4.93 mm left there, 7.6 A); its 3V3 end is a scripted pre-route.
- R19 / R20: 4.7k -> 10k (I2C bus ~1.05 k with the module pull-ups).
- SMD_PAD_VIA = (0.8, 0.3) for the SMD_GND_VIAS; net_via() takes the via position;
  stitching vias stay GND_VIA (0.8 / 0.4).
- DRC_RULES: JLCPCB 4-layer minimums (annular ring, plated / non-plated hole, hole to hole,
  copper to edge, silk line / text stroke, silk to mask), each checked against a deliberate
  violation; copper to edge stays at KiCad's 0.5 mm.
- Regenerated schematic, board, routing, fab package and board_cad.json; docs and tests updated.

Co-Authored-By: Claude Opus 5.5 <noreply@anthropic.com>
Parts:
- added C4, C5: 100nF, Capacitor_SMD:C_0805_2012Metric, symbol Device:C
- added D2: SS14, Diode_SMD:D_SMA, symbol Diode:SS14
- added R24, R25: 4.7k, Resistor_SMD:R_0805_2012Metric, symbol Device:R
- added R26: 10k, Resistor_SMD:R_0805_2012Metric, symbol Device:R
- R19, R20: value 4.7k -> 10k
Connections:
- net 3V3: now also R26.2
- net 5V: now also D2.2 (A)
- net ARM: now also R26.1
- net GND: now also C4.2, C5.2
- net L_CS: now also R24.1; no longer U1B.9 (Pin_9)
- net R_CS: now also R25.1; no longer U1B.7 (Pin_7)
- net VSYS: now reaches U1B.2 (Pin_2)
- net VSYS: now also D2.1 (K)
- new net L_CS_ADC: C4.1, R24.2, U1B.9 (Pin_9)
- new net R_CS_ADC: C5.1, R25.2, U1B.7 (Pin_7)
- no-connect marks 15 -> 14
Other:
- moved on the sheet: D1, F1, F2, H1, H2, H3, H4, H5, H6, J1, J10, J11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
